Commit message: Update six_dof_arm.urdf

File: urdf/six_dof_arm.urdf (robot description, URDF)
Before this commit: robot six_dof_arm, 7 links, 6 joints
Links:
- removed link link_6
- added link clawl; collision mesh filename=package://six_dof_arm/meshes/clawl.stl scale=0.0001 0.0001 0.0001; visual mesh filename=package://six_dof_arm/meshes/clawl.stl scale=0.0001 0.0001 0.0001
- added link clawr; collision mesh filename=package://six_dof_arm/meshes/clawr.stl scale=0.0001 0.0001 0.0001; visual mesh filename=package://six_dof_arm/meshes/clawr.stl scale=0.0001 0.0001 0.0001
Joints:
- removed joint joint_6
- added joint joint_7: type revolute, parent link_5, child clawr, origin xyz=0.011 0.034 0 rpy=0 0 -0.31, axis 0 0 1, limit lower=-0.5 upper=0.0 effort=1000.0 velocity=1.0
- added joint joint_8: type revolute, parent link_5, child clawl, origin xyz=-0.016 0.030 0 rpy=0 0 0.22, axis 0 0 1, limit lower=0 upper=-0.5 effort=1000.0 velocity=1.0, mimic joint=joint_7 multiplier=-1 offset=0

Commit message: Update six_dof_arm.urdf

File: urdf/six_dof_arm.urdf (robot description, URDF)
Before this commit: robot six_dof_arm, 8 links, 7 joints
Joints:
- joint joint_7: origin xyz=0.011 0.034 0 rpy=0 0 -0.31 -> xyz=0.011 0.034 0.005 rpy=0 0 -0.31
- joint joint_8: limit lower=0 upper=-0.5 effort=1000.0 velocity=1.0 -> lower=0 upper=0.5 effort=1000.0 velocity=1.0

Commit message: Update six_dof_arm.urdf

File: urdf/six_dof_arm.urdf (robot description, URDF)
Before this commit: robot six_dof_arm, 8 links, 7 joints
Joints:
- joint joint_1: limit lower=-2.355 upper=2.355 effort=20 velocity=3 -> lower=-1.57 upper=1.57 effort=20 velocity=3; origin xyz=0.0575229584695751 0 0.052 rpy=1.5707963267949 0 1.5707963267949 -> xyz=0.0575229584695751 0 0.052 rpy=1.5707963267949 0 -1.5707963267949
- joint joint_2: limit lower=-0.785 upper=1.57 effort=20 velocity=3 -> lower=-2.26 upper=1.04 effort=20 velocity=3
- joint joint_3: limit lower=-2.26 upper=2.26 effort=20 velocity=3 -> lower=-2.53 upper=0.61 effort=20 velocity=3
- joint joint_4: limit lower=-2.26 upper=2.26 effort=20 velocity=3 -> lower=-0.87 upper=1.79 effort=20 velocity=3
- joint joint_5: limit lower=-2.26 upper=2.26 effort=20 velocity=3 -> lower=-1.57 upper=1.57 effort=20 velocity=3
- joint joint_7: limit lower=-0.5 upper=0.0 effort=1000.0 velocity=1.0 -> lower=-1.22 upper=0 effort=1000.0 velocity=1.0
- joint joint_8: limit lower=0 upper=0.5 effort=1000.0 velocity=1.0 -> lower=-1.22 upper=0 effort=1000.0 velocity=1.0

Commit message: Update six_dof_arm.urdf

File: urdf/six_dof_arm.urdf (robot description, URDF)
Before this commit: robot six_dof_arm, 8 links, 7 joints
Joints:
- joint joint_7: limit lower=-1.22 upper=0 effort=1000.0 velocity=1.0 -> lower=-0.61 upper=0 effort=1000.0 velocity=5.0
- joint joint_8: limit lower=-1.22 upper=0 effort=1000.0 velocity=1.0 -> lower=-0.61 upper=0 effort=1000.0 velocity=5.0

Commit message: Update six_dof_arm.urdf

File: urdf/six_dof_arm.urdf (robot description, URDF)
Before this commit: robot six_dof_arm, 8 links, 7 joints
Joints:
- joint joint_4: limit lower=-0.87 upper=1.79 effort=20 velocity=3 -> lower=-0.87 upper=1.74 effort=20 velocity=3

Commit message: Update six_dof_arm.urdf

File: urdf/six_dof_arm.urdf (robot description, URDF)
Before this commit: robot six_dof_arm, 8 links, 7 joints
Joints:
- joint joint_1: limit lower=-1.57 upper=1.57 effort=20 velocity=3 -> lower=-1.57 upper=1.57 effort=10 velocity=3
- joint joint_2: limit lower=-2.26 upper=1.04 effort=20 velocity=3 -> lower=-2.26 upper=1.04 effort=10 velocity=3
- joint joint_3: limit lower=-2.53 upper=0.61 effort=20 velocity=3 -> lower=-2.53 upper=0.61 effort=10 velocity=3
- joint joint_4: limit lower=-0.87 upper=1.74 effort=20 velocity=3 -> lower=-0.87 upper=1.74 effort=10 velocity=3
- joint joint_5: limit lower=-1.57 upper=1.57 effort=20 velocity=3 -> lower=-1.57 upper=1.57 effort=10 velocity=3
- joint joint_7: limit lower=-0.61 upper=0 effort=1000.0 velocity=5.0 -> lower=-0.61 upper=0 effort=10.0 velocity=5.0
- joint joint_8: limit lower=-0.61 upper=0 effort=1000.0 velocity=5.0 -> lower=-0.61 upper=0 effort=10.0 velocity=5.0

Commit message: Update six_dof_arm.urdf

File: urdf/six_dof_arm.urdf (robot description, URDF)
Before this commit: robot six_dof_arm, 8 links, 7 joints
Links:
- added link world
Joints:
- added joint world_to_arm: type fixed, parent world, child base_link, origin xyz=0 0 0 rpy=0 0 0

Commit message: Update six_dof_arm.urdf

File: urdf/six_dof_arm.urdf (robot description, URDF)
Before this commit: robot six_dof_arm, 9 links, 8 joints
Joints:
- joint joint_1: limit lower=-1.57 upper=1.57 effort=10 velocity=3 -> lower=-1.57 upper=1.57 effort=20 velocity=3
- joint joint_2: limit lower=-2.26 upper=1.04 effort=10 velocity=3 -> lower=-2.26 upper=1.04 effort=20 velocity=3
- joint joint_3: limit lower=-2.53 upper=0.61 effort=10 velocity=3 -> lower=-2.53 upper=0.61 effort=20 velocity=3
- joint joint_4: limit lower=-0.87 upper=1.74 effort=10 velocity=3 -> lower=-0.87 upper=1.74 effort=20 velocity=3
- joint joint_5: limit lower=-1.57 upper=1.57 effort=10 velocity=3 -> lower=-1.57 upper=1.57 effort=20 velocity=3
- joint joint_7: limit lower=-0.61 upper=0 effort=10.0 velocity=5.0 -> lower=-0.61 upper=0 effort=100.0 velocity=5.0
- joint joint_8: limit lower=-0.61 upper=0 effort=10.0 velocity=5.0 -> lower=-0.61 upper=0 effort=100.0 velocity=5.0
- joint world_to_arm: origin xyz=0 0 0 rpy=0 0 0 -> xyz=0 0 0.01 rpy=0 0 0

Commit message: Update six_dof_arm.urdf

File: urdf/six_dof_arm.urdf (robot description, URDF)
Before this commit: robot six_dof_arm, 9 links, 8 joints
Links:
- removed link clawl
- removed link clawr
- added link camera_link, mass 1e-5; collision box size=0.2 0.2 0.2; visual box size=0.2 0.2 0.2
- added link link_6, mass 0.0123483072583734; collision mesh filename=package://six_dof_arm/meshes/link_6.STL; visual mesh filename=package://six_dof_arm/meshes/link_6.STL
Joints:
- removed joint joint_7
- removed joint joint_8
- added joint camera_joint: type fixed, parent world, child camera_link, origin xyz=0 0 0.8 rpy=0 0 0, axis 0 1 0
- added joint joint_6: type revolute, parent link_5, child link_6, origin xyz=-0.0140033661195784 0.0319999999999998 0.00298424820030765 rpy=3.14159265358979 0 0, axis 0.00112499294844597 0 0.999999367195233, limit lower=-2.26 upper=2.26 effort=20 velocity=3
- joint joint_1: limit lower=-1.57 upper=1.57 effort=20 velocity=3 -> lower=-2.355 upper=2.355 effort=20 velocity=3; origin xyz=0.0575229584695751 0 0.052 rpy=1.5707963267949 0 -1.5707963267949 -> xyz=0.0575229584695751 0 0.052 rpy=1.5707963267949 0 1.5707963267949
- joint joint_2: limit lower=-2.26 upper=1.04 effort=20 velocity=3 -> lower=-0.785 upper=1.57 effort=20 velocity=3
- joint joint_3: limit lower=-2.53 upper=0.61 effort=20 velocity=3 -> lower=-2.26 upper=2.26 effort=20 velocity=3
- joint joint_4: limit lower=-0.87 upper=1.74 effort=20 velocity=3 -> lower=-2.26 upper=2.26 effort=20 velocity=3
- joint joint_5: limit lower=-1.57 upper=1.57 effort=20 velocity=3 -> lower=-2.26 upper=2.26 effort=20 velocity=3
